File: eagle/boards/TB6560AHQ_rev2/schematic.brd (EAGLE design)
At the start: 58.4 x 60.6 mm, 24 parts, among them IC1 7805TV

Commit message: update
Parts:
- added H1: MOUNT-HOLE4.1, holes:4,1
- C7: device rcl:E2,5-6E -> rcl:E2,5-5
- moved C7 38.2 mm to (118.1, 59.7), turned to 270 degrees
Routing:
- net GND: track 279.2 -> 347.1 mm, vias 4 -> 8
- net VCC: track 222.8 -> 210.4 mm, vias 2 -> 1
- net +24V: track 210.2 -> 212.2 mm
