File: eagle/boards/TB6560AHQ_rev2/schematic.sch (EAGLE design)
At the start: 24 parts, among them IC1 7805TV

Commit message: update
Parts:
- added H1: MOUNT-HOLE4.1, holes:MOUNT-HOLE4.1
- C7: device rcl:CPOL-EUE2,5-6E -> rcl:CPOL-EUE2.5-5
Changed lines of the file:
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@@
 <part name="C5" library="rcl" deviceset="C-EU" device="C0805K" value=".1"/>
 <part name="IC1" library="linear" deviceset="78*" device="TV" technology="05"/>
-<part name="C7" library="rcl" deviceset="CPOL-EU" device="E2,5-6E" value="10uF"/>
+<part name="C7" library="rcl" deviceset="CPOL-EU" device="E2.5-5" value="10uF"/>
 <part name="C8" library="rcl" deviceset="CPOL-EU" device="E2.5-5" value="47uF 50V"/>
 <part name="P+5" library="supply1" deviceset="VCC" device=""/>
@@
 <part name="C6" library="rcl" deviceset="CPOL-EU" device="E2.5-5" value="25uF"/>
 <part name="GND7" library="supply1" deviceset="GND" device=""/>
+<part name="H1" library="holes" deviceset="MOUNT-HOLE" device="4.1"/>
 </parts>
 <sheets>
@@
 <instance part="C6" gate="G$1" x="-63.5" y="68.58"/>
 <instance part="GND7" gate="1" x="-63.5" y="58.42"/>
+<instance part="H1" gate="G$1" x="-129.54" y="-27.94"/>
 </instances>
 <busses>
@@
 <segment>
 <pinref part="U$1" gate="G$1" pin="M2"/>
-<wire x1="-25.4" y1="2.54" x2="-53.34" y2="2.54" width="0.1524" layer="91"/>
-<wire x1="-53.34" y1="2.54" x2="-53.34" y2="0" width="0.1524" layer="91"/>
+<wire x1="-25.4" y1="2.54" x2="-43.18" y2="2.54" width="0.1524" layer="91"/>
+<wire x1="-43.18" y1="2.54" x2="-43.18" y2="0" width="0.1524" layer="91"/>
 <pinref part="JP1" gate="A" pin="2"/>
-<wire x1="-53.34" y1="0" x2="-60.96" y2="0" width="0.1524" layer="91"/>
-</segment>
-</net>
+<wire x1="-43.18" y1="0" x2="-60.96" y2="0" width="0.1524" layer="91"/>
+</segment>
+</net>
