File: eagle/boards/SIM900/sim900.brd (EAGLE design)
At the start: 50.8 x 63.2 mm, 24 parts, among them IC1 SIM900, X1 SIMLOCK-C707_10M006_512_2

Commit message: update sim900
Parts:
- moved R3 11.7 mm to (45.7, 30.5), flipped to the bottom, turned to 180 degrees
- moved T1 9.92 mm to (45.7, 35.6), flipped to the bottom
- moved R1 9.16 mm to (45.7, 39.4), flipped to the bottom, turned to 0 degrees
- moved T2 7.73 mm to (45.7, 43.2), flipped to the bottom
- moved R2 7.62 mm to (45.7, 24.1)
- moved C1 6.84 mm to (45.7, 50.8), flipped to the bottom
- moved R8 6.48 mm to (68.6, 24.1), flipped to the bottom
- moved C2 6.35 mm to (68.6, 53.3), flipped to the bottom
- moved R5 6.35 mm to (68.6, 45.7), flipped to the bottom
- moved R6 6.35 mm to (68.6, 40.6), flipped to the bottom
- moved R7 6.35 mm to (68.6, 30.5), flipped to the bottom
- moved T3 6.35 mm to (68.6, 35.6), flipped to the bottom, turned to 90 degrees
- moved R4 6.35 mm to (45.7, 19.1)
- moved C3 4.02 mm to (67.3, 59.7)
- moved C5 2.54 mm to (64.8, 50.8)
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Connections:
- net SCL: now also U$1.B4; no longer U$1.B2
- net SDA: now also U$1.B2; no longer U$1.B4
Routing:
- net GND: track 75.8 -> 243.2 mm, vias 2 -> 6
- net VCC: track 0.00 -> 55.8 mm, vias 0 -> 1
- net TXD: track 0.00 -> 48.6 mm, vias 0 -> 1
- net RXD: track 0.00 -> 48.0 mm, vias 0 -> 1
- net N$15: track 0.00 -> 43.4 mm, vias 0 -> 1
- net N$6: track 0.00 -> 41.2 mm, vias 0 -> 1
- net SCL: track 0.00 -> 35.3 mm, vias 0 -> 1
- net SDA: track 0.00 -> 32.8 mm, vias 0 -> 1
- net LINEIN_R: track 0.00 -> 31.8 mm, vias 0 -> 1
- net LINEIN_L: track 0.00 -> 30.9 mm, vias 0 -> 3
- net VRTC: track 0.00 -> 26.9 mm
- net SPK1N: track 0.00 -> 26.6 mm
- net ADC: track 0.00 -> 26.3 mm
- net SPK1P: track 0.00 -> 25.9 mm
- net MIC1N: track 0.00 -> 25.2 mm
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Other:
- board size 50.8 x 63.2 mm -> 39.4 x 57.5 mm

Commit message: update
Parts:
- C5: device rcl:C0805K -> rcl:C1206K
- moved U$1 5.00 mm to (55.9, 12.6)
- moved R10 3.27 mm to (59.8, 21.0), turned to 225 degrees
- moved R8 2.54 mm to (71.1, 24.1)
- moved R4 2.54 mm to (45.7, 21.6)
- moved R3 2.13 mm to (43.8, 31.4), turned to 270 degrees
- moved X1 2.00 mm to (57.1, 38.8)
- moved R11 1.00 mm to (58.4, 54.3)
- moved R9 1.00 mm to (52.1, 54.3)
- moved R12 0.63 mm to (63.5, 19.7)
Connections:
- net RST renamed 456
- removed net LED: U$1.T3
- removed net VCC: C1.+, C2.+, C3.1, C4.1, R8.2
- new net 123: U$1.T13
- net ADC: now also U$1.T3; no longer U$1.T7
- net MIC1N: now also U$1.T9; no longer U$1.T13
- net MIC1P: now also U$1.T11; no longer U$1.T15
- net ON_OFF: now also U$1.T15; no longer U$1.T1
- net SPK1N: now also U$1.T5; no longer U$1.T9
- net SPK1P: now also U$1.T7; no longer U$1.T11
- net VBAT: now also C1.+, C2.+, C3.1, C4.1, R8.2
- net VRTC: now also U$1.T1; no longer U$1.T5
Routing:
- net VBAT: track 4.54 -> 149.7 mm, vias 0 -> 3
- net VCC: track 55.8 -> 0.00 mm, vias 1 -> 0
- net N$12: track 4.32 -> 42.7 mm, vias 0 -> 1
- net ON_OFF: track 0.00 -> 27.9 mm, vias 0 -> 1
- net N$6: track 41.2 -> 61.0 mm
- net GND: track 243.2 -> 261.6 mm
- net N$9: track 0.00 -> 16.5 mm, vias 0 -> 1
- net LINEIN_R: track 31.8 -> 23.6 mm
- net TXD: track 48.6 -> 41.6 mm
- net N$5: track 20.4 -> 14.2 mm
- net LINEIN_L: track 30.9 -> 34.9 mm
- net RXD: track 48.0 -> 44.2 mm
- net SDA: track 32.8 -> 29.3 mm
- net RESET: track 20.9 -> 17.7 mm
- net MIC1N: track 25.2 -> 22.3 mm
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- added copper zone on layer 1, net N$17
- added copper zone on layer 16, net N$18
Other:
- board size 39.4 x 57.5 mm -> 34 x 53 mm
