File: eagle/boards/SIM900/sim900.sch (EAGLE design)
At the start: 24 parts, among them IC1 SIM900, X1 SIMLOCK-C707_10M006_512_2

Commit message: update sim900
Connections:
- net SCL: now also U$1.C4; no longer U$1.C2
- net SDA: now also U$1.C2; no longer U$1.C4
Changed lines of the file:
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@@
 <part name="GND13" library="supply1" deviceset="GND" device=""/>
 <part name="R12" library="rcl" deviceset="R-EU_" device="R0805"/>
+<part name="P+3" library="supply1" deviceset="VCC" device=""/>
 </parts>
 <sheets>
@@
 <instance part="GND13" gate="1" x="2.54" y="-88.9"/>
 <instance part="R12" gate="G$1" x="7.62" y="-60.96" rot="R270"/>
+<instance part="P+3" gate="VCC" x="142.24" y="45.72"/>
 </instances>
 <busses>
@@
 </segment>
 <segment>
+<pinref part="U$1" gate="G$1" pin="C4"/>
+<wire x1="109.22" y1="30.48" x2="109.22" y2="20.32" width="0.1524" layer="91"/>
+<label x="109.22" y="20.32" size="1.778" layer="95" rot="R90"/>
+</segment>
+</net>
+<net name="SDA" class="0">
+<segment>
+<pinref part="IC1" gate="G$1" pin="SDA"/>
+<wire x1="40.64" y1="-15.24" x2="48.26" y2="-15.24" width="0.1524" layer="91"/>
+<label x="43.18" y="-15.24" size="1.778" layer="95"/>
+</segment>
+<segment>
 <pinref part="U$1" gate="G$1" pin="C2"/>
 <wire x1="106.68" y1="30.48" x2="106.68" y2="20.32" width="0.1524" layer="91"/>
 <label x="106.68" y="20.32" size="1.778" layer="95" rot="R90"/>
-</segment>
-</net>
-<net name="SDA" class="0">
-<segment>
-<pinref part="IC1" gate="G$1" pin="SDA"/>
-<wire x1="40.64" y1="-15.24" x2="48.26" y2="-15.24" width="0.1524" layer="91"/>
-<label x="43.18" y="-15.24" size="1.778" layer="95"/>
-</segment>
-<segment>
-<pinref part="U$1" gate="G$1" pin="C4"/>
-<wire x1="109.22" y1="30.48" x2="109.22" y2="20.32" width="0.1524" layer="91"/>
-<label x="109.22" y="20.32" size="1.778" layer="95" rot="R90"/>
 </segment>
 </net>
@@
 <wire x1="127" y1="40.64" x2="129.54" y2="40.64" width="0.1524" layer="91"/>
 <junction x="129.54" y="40.64"/>
-<wire x1="129.54" y1="40.64" x2="139.7" y2="40.64" width="0.1524" layer="91"/>
-</segment>
-</net>
+</segment>
+<segment>
+<pinref part="P+3" gate="VCC" pin="VCC"/>
+<wire x1="142.24" y1="43.18" x2="142.24" y2="38.1" width="0.1524" layer="91"/>
+<wire x1="142.24" y1="38.1" x2="157.48" y2="38.1" width="0.1524" layer="91"/>
+</segment>
+</net>

Commit message: update
Parts:
- C5: device rcl:C-EUC0805K -> rcl:C-EUC1206K
Connections:
- net RST renamed 456
- removed net LED: U$1.C3
- removed net VCC: C1.+, C2.+, C3.1, C4.1, R8.2
- new net 123: U$1.C13
- net ADC: now also U$1.C3; no longer U$1.C7
- net MIC1N: now also U$1.C9; no longer U$1.C13
- net MIC1P: now also U$1.C11; no longer U$1.C15
- net ON_OFF: now also U$1.C15; no longer U$1.C1
- net SPK1N: now also U$1.C5; no longer U$1.C9
- net SPK1P: now also U$1.C7; no longer U$1.C11
- net VBAT: now also C1.+, C2.+, C3.1, C4.1, R8.2
- net VRTC: now also U$1.C1; no longer U$1.C5
Other:
- moved on the sheet: C1, C2, C3, C4
