File: eagle/boards/OpenLRS/kolrs868_rx.brd (EAGLE design)
At the start: 35.6 x 54.6 mm, 41 parts, among them IC1 LE33CD, J1 AVR_SPI_PRG_6PTH, Q1 16MHz, U1 ATMEGA328-AU, X2 BU-SMA-V

Commit message: OpenLRS rx board routed
Parts:
- moved C6 2.40 mm to (17.8, 38.0)
- moved R11 2.03 mm to (21.0, 38.0)
- moved C9 1.69 mm to (5.26, 17.3)
- moved IC1 1.27 mm to (32.6, 8.74)
- moved C5 1.13 mm to (12.2, 25.3)
- moved LED2 0.87 mm to (26.6, 42.7)
- moved C8 0.84 mm to (5.27, 28.0)
- moved R12 0.62 mm to (24.1, 38.0)
- moved LED1 0.60 mm to (23.4, 42.7)
- moved R13 0.52 mm to (27.3, 38.0)
- moved X2 0.10 mm to (6.45, 48.3)
Routing:
- net GND: track 525.3 -> 22.6 mm, vias 1 -> 125
- net VCC: track 108.4 -> 122.4 mm, vias 3 -> 4
- net RX: track 24.8 -> 31.8 mm, vias 2 -> 0
- net D13: track 39.6 -> 33.1 mm
- net DTR: track 26.2 -> 21.4 mm
- net A3: track 14.7 -> 10.5 mm
- net SDA: track 25.1 -> 21.0 mm, vias 0 -> 1
- net D11: track 26.2 -> 22.1 mm, vias 2 -> 0
- net N$24: track 8.51 -> 12.6 mm
- net D7: track 10.0 -> 14.0 mm, vias 0 -> 2
- net A1/SDI: track 24.1 -> 27.5 mm
- net D2/NIRQ: track 25.8 -> 28.8 mm
- net SCL: track 25.6 -> 22.7 mm, vias 0 -> 1
- net A2/SCLK: track 24.0 -> 26.1 mm
- net N$6: track 17.8 -> 16.0 mm
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- added copper zone on layer 1, net GND
- added copper zone on layer 16, net GND
Other:
- board size 35.6 x 54.6 mm -> 37.1 x 56.2 mm
- board text added: "KOLRS RX 1.1 ROMIX.LAB 23BP"
- board text added: "romix.lab"
- board text removed: "433"
- board text removed: "868"
- board text removed: "KOLRS RX 1.1"
