File: eagle/boards/OpenLRS/kolrs868_rx.sch (EAGLE design)
At the start: 41 parts, among them IC1 LE33CD, J1 AVR_SPI_PRG_6PTH, Q1 16MHz, U1 ATMEGA328-AU, X2 BU-SMA-V

Commit message: OpenLRS rx board routed
Other:
- note added: "(c) romix.lab"
Changed lines of the file:
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@@
 <?xml version="1.0" encoding="utf-8"?>
 <!DOCTYPE eagle SYSTEM "eagle.dtd">
-<eagle version="6.5.0">
+<eagle version="6.4">
 <drawing>
 <settings>
@@
 <text x="55.88" y="-22.86" size="2.54" layer="94">(c) Flytron</text>
 <text x="55.88" y="-27.94" size="2.54" layer="94">(c) kolin</text>
+<text x="55.88" y="-33.02" size="2.54" layer="94">(c) romix.lab</text>
 </plain>
 <instances>
