File: eagle/boards/ATMega128RFR2-Module/module.sch (EAGLE design)
At the start: 2 parts, among them U1 ATMEGA256RFR2

Commit message: Schematic work started
Parts:
- added C1, C2, C3, C4: 1uF, rcl:C-EUC0805K
- added Q1: 16MHz, crystal:86SMX
Connections:
- new net +3V3: C2.1, C4.1, U1.DEVDD@23, U1.DEVDD@34, U1.DEVDD@44, U1.DEVDD@54, U1.EVDD
- new net ANT: F1.UNBAL
- new net GND: U1.AVSS@58, U1.AVSS@61, U1.AVSS_RFN, U1.AVSS_RFP, U1.DVSS@20, U1.DVSS@24, U1.DVSS@35, U1.DVSS@45, U1.DVSS@55
- new net N$1: C3.1, U1.DVDD@21, U1.DVDD@22
- new net N$2: C1.1, U1.AVDD
- new net N$3: Q1.2, U1.XTAL1
- new net N$4: Q1.1, U1.XTAL2
- new net RFN: F1.BAL1, U1.RFN
- new net RFP: F1.BAL2, U1.RFP
- new net RSTN: U1.RSTN
Changed lines of the file:
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@@
 <part name="U1" library="RFR2" deviceset="ATMEGA256RFR2" device=""/>
 <part name="F1" library="RFR2" deviceset="2450BM15A0002" device=""/>
+<part name="Q1" library="crystal" deviceset="86SMX" device="" value="16MHz"/>
+<part name="C1" library="rcl" deviceset="C-EU" device="C0805K" value="1uF"/>
+<part name="C2" library="rcl" deviceset="C-EU" device="C0805K" value="1uF"/>
+<part name="GND1" library="supply1" deviceset="GND" device=""/>
+<part name="GND2" library="supply1" deviceset="GND" device=""/>
+<part name="GND3" library="supply1" deviceset="GND" device=""/>
+<part name="GND4" library="supply1" deviceset="GND" device=""/>
+<part name="+3V1" library="supply1" deviceset="+3V3" device=""/>
+<part name="C3" library="rcl" deviceset="C-EU" device="C0805K" value="1uF"/>
+<part name="C4" library="rcl" deviceset="C-EU" device="C0805K" value="1uF"/>
+<part name="+3V2" library="supply1" deviceset="+3V3" device=""/>
 </parts>
 <sheets>
@@
 <instance part="U1" gate="G$1" x="0" y="0"/>
 <instance part="F1" gate="G$1" x="-17.78" y="76.2"/>
+<instance part="Q1" gate="G$1" x="-43.18" y="-2.54" rot="R90"/>
+<instance part="C1" gate="G$1" x="-50.8" y="20.32"/>
+<instance part="C2" gate="G$1" x="-66.04" y="20.32"/>
+<instance part="GND1" gate="1" x="-33.02" y="-55.88"/>
+<instance part="GND2" gate="1" x="-40.64" y="-55.88"/>
+<instance part="GND3" gate="1" x="-48.26" y="-55.88"/>
+<instance part="GND4" gate="1" x="-48.26" y="10.16"/>
+<instance part="+3V1" gate="G$1" x="-53.34" y="45.72"/>
+<instance part="C3" gate="G$1" x="-43.18" y="20.32"/>
+<instance part="C4" gate="G$1" x="-58.42" y="20.32"/>
+<instance part="+3V2" gate="G$1" x="-63.5" y="35.56"/>
 </instances>
 <busses>
 </busses>
 <nets>
+<net name="RFN" class="0">
+<segment>
+<pinref part="F1" gate="G$1" pin="BAL1"/>
+<wire x1="-27.94" y1="81.28" x2="-35.56" y2="81.28" width="0.1524" layer="91"/>
+<label x="-35.56" y="81.28" size="1.778" layer="95"/>
+</segment>
+<segment>
+<pinref part="U1" gate="G$1" pin="RFN"/>
+<wire x1="-27.94" y1="5.08" x2="-35.56" y2="5.08" width="0.1524" layer="91"/>
+<label x="-35.56" y="5.08" size="1.778" layer="95"/>
+</segment>
+</net>
+<net name="RFP" class="0">
+<segment>
+<pinref part="F1" gate="G$1" pin="BAL2"/>
+<wire x1="-27.94" y1="76.2" x2="-35.56" y2="76.2" width="0.1524" layer="91"/>
+<label x="-35.56" y="76.2" size="1.778" layer="95"/>
+</segment>
+<segment>
+<pinref part="U1" gate="G$1" pin="RFP"/>
+<wire x1="-27.94" y1="7.62" x2="-35.56" y2="7.62" width="0.1524" layer="91"/>
+<label x="-35.56" y="7.62" size="1.778" layer="95"/>
+</segment>
+</net>
+<net name="ANT" class="0">
+<segment>
+<pinref part="F1" gate="G$1" pin="UNBAL"/>
+<wire x1="-7.62" y1="78.74" x2="0" y2="78.74" width="0.1524" layer="91"/>
+<label x="-5.08" y="78.74" size="1.778" layer="95"/>
+</segment>
+</net>
+<net name="GND" class="0">
+<segment>
+<pinref part="GND1" gate="1" pin="GND"/>
+<wire x1="-33.02" y1="-53.34" x2="-33.02" y2="-50.8" width="0.1524" layer="91"/>
+<pinref part="U1" gate="G$1" pin="AVSS@61"/>
+<wire x1="-33.02" y1="-50.8" x2="-27.94" y2="-50.8" width="0.1524" layer="91"/>
+<pinref part="U1" gate="G$1" pin="AVSS@58"/>
+<wire x1="-27.94" y1="-48.26" x2="-33.02" y2="-48.26" width="0.1524" layer="91"/>
+<wire x1="-33.02" y1="-48.26" x2="-33.02" y2="-50.8" width="0.1524" layer="91"/>
+<junction x="-33.02" y="-50.8"/>
+</segment>
+<segment>
+<pinref part="GND2" gate="1" pin="GND"/>
+<wire x1="-40.64" y1="-53.34" x2="-40.64" y2="-45.72" width="0.1524" layer="91"/>
+<pinref part="U1" gate="G$1" pin="DVSS@24"/>
+<wire x1="-27.94" y1="-38.1" x2="-33.02" y2="-38.1" width="0.1524" layer="91"/>
+<wire x1="-33.02" y1="-38.1" x2="-33.02" y2="-40.64" width="0.1524" layer="91"/>
+<pinref part="U1" gate="G$1" pin="DVSS@35"/>
+<wire x1="-33.02" y1="-40.64" x2="-27.94" y2="-40.64" width="0.1524" layer="91"/>
+<wire x1="-33.02" y1="-40.64" x2="-33.02" y2="-43.18" width="0.1524" layer="91"/>
+<junction x="-33.02" y="-40.64"/>
+<pinref part="U1" gate="G$1" pin="DVSS@45"/>
+<wire x1="-33.02" y1="-43.18" x2="-27.94" y2="-43.18" width="0.1524" layer="91"/>
+<pinref part="U1" gate="G$1" pin="DVSS@55"/>
+<wire x1="-27.94" y1="-45.72" x2="-33.02" y2="-45.72" width="0.1524" layer="91"/>
+<wire x1="-33.02" y1="-45.72" x2="-33.02" y2="-43.18" width="0.1524" layer="91"/>
+<junction x="-33.02" y="-43.18"/>
+<wire x1="-33.02" y1="-38.1" x2="-33.02" y2="-35.56" width="0.1524" layer="91"/>
+<junction x="-33.02" y="-38.1"/>
+<pinref part="U1" gate="G$1" pin="DVSS@20"/>
+<wire x1="-33.02" y1="-35.56" x2="-27.94" y2="-35.56" width="0.1524" layer="91"/>
+<wire x1="-40.64" y1="-45.72" x2="-33.02" y2="-45.72" width="0.1524" layer="91"/>
+<junction x="-33.02" y="-45.72"/>
+</segment>
+<segment>
+<pinref part="GND3" gate="1" pin="GND"/>
+<wire x1="-48.26" y1="-53.34" x2="-48.26" y2="-33.02" width="0.1524" layer="91"/>
+<pinref part="U1" gate="G$1" pin="AVSS_RFN"/>
+<wire x1="-27.94" y1="-33.02" x2="-33.02" y2="-33.02" width="0.1524" layer="91"/>
+<wire x1="-33.02" y1="-33.02" x2="-33.02" y2="-30.48" width="0.1524" layer="91"/>
+<pinref part="U1" gate="G$1" pin="AVSS_RFP"/>
+<wire x1="-33.02" y1="-30.48" x2="-27.94" y2="-30.48" width="0.1524" layer="91"/>
+<wire x1="-48.26" y1="-33.02" x2="-33.02" y2="-33.02" width="0.1524" layer="91"/>
+<junction x="-33.02" y="-33.02"/>
+</segment>
+</net>
+<net name="N$2" class="0">
+<segment>
+<pinref part="U1" gate="G$1" pin="AVDD"/>
+<wire x1="-27.94" y1="27.94" x2="-43.18" y2="27.94" width="0.1524" layer="91"/>
+<pinref part="C1" gate="G$1" pin="1"/>
+<wire x1="-43.18" y1="27.94" x2="-50.8" y2="22.86" width="0.1524" layer="91"/>
+</segment>
+</net>
+<net name="+3V3" class="0">
+<segment>
+<pinref part="U1" gate="G$1" pin="EVDD"/>
+<pinref part="C2" gate="G$1" pin="1"/>
+<wire x1="-27.94" y1="40.64" x2="-53.34" y2="40.64" width="0.1524" layer="91"/>
+<wire x1="-53.34" y1="40.64" x2="-66.04" y2="22.86" width="0.1524" layer="91"/>
+<pinref part="+3V1" gate="G$1" pin="+3V3"/>
+<wire x1="-53.34" y1="40.64" x2="-53.34" y2="43.18" width="0.1524" layer="91"/>
+<junction x="-53.34" y="40.64"/>
+</segment>
+<segment>
+<pinref part="U1" gate="G$1" pin="DEVDD@23"/>
+<wire x1="-27.94" y1="38.1" x2="-30.48" y2="38.1" width="0.1524" layer="91"/>
+<wire x1="-30.48" y1="38.1" x2="-30.48" y2="35.56" width="0.1524" layer="91"/>
+<pinref part="U1" gate="G$1" pin="DEVDD@34"/>
+<wire x1="-30.48" y1="35.56" x2="-27.94" y2="35.56" width="0.1524" layer="91"/>
+<wire x1="-30.48" y1="35.56" x2="-30.48" y2="33.02" width="0.1524" layer="91"/>
+<junction x="-30.48" y="35.56"/>
+<pinref part="U1" gate="G$1" pin="DEVDD@44"/>
+<wire x1="-30.48" y1="33.02" x2="-27.94" y2="33.02" width="0.1524" layer="91"/>
+<wire x1="-30.48" y1="33.02" x2="-30.48" y2="30.48" width="0.1524" layer="91"/>
+<junction x="-30.48" y="33.02"/>
+<pinref part="U1" gate="G$1" pin="DEVDD@54"/>
+<wire x1="-30.48" y1="30.48" x2="-27.94" y2="30.48" width="0.1524" layer="91"/>
+<pinref part="C4" gate="G$1" pin="1"/>
+<wire x1="-30.48" y1="30.48" x2="-63.5" y2="30.48" width="0.1524" layer="91"/>
+<wire x1="-63.5" y1="30.48" x2="-58.42" y2="22.86" width="0.1524" layer="91"/>
+<junction x="-30.48" y="30.48"/>
+<pinref part="+3V2" gate="G$1" pin="+3V3"/>
+<wire x1="-63.5" y1="30.48" x2="-63.5" y2="33.02" width="0.1524" layer="91"/>
+<junction x="-63.5" y="30.48"/>
+</segment>
+</net>
+<net name="N$1" class="0">
+<segment>
+<pinref part="U1" gate="G$1" pin="DVDD@22"/>
+<wire x1="-27.94" y1="22.86" x2="-33.02" y2="22.86" width="0.1524" layer="91"/>
+<wire x1="-33.02" y1="22.86" x2="-33.02" y2="25.4" width="0.1524" layer="91"/>
+<pinref part="U1" gate="G$1" pin="DVDD@21"/>
+<wire x1="-33.02" y1="25.4" x2="-27.94" y2="25.4" width="0.1524" layer="91"/>
+<pinref part="C3" gate="G$1" pin="1"/>
+<wire x1="-33.02" y1="25.4" x2="-38.1" y2="25.4" width="0.1524" layer="91"/>
+<wire x1="-38.1" y1="25.4" x2="-43.18" y2="22.86" width="0.1524" layer="91"/>
+<junction x="-33.02" y="25.4"/>
+</segment>
+</net>
+<net name="RSTN" class="0">
+<segment>
+<pinref part="U1" gate="G$1" pin="RSTN"/>
+<wire x1="-27.94" y1="15.24" x2="-35.56" y2="15.24" width="0.1524" layer="91"/>
+<label x="-35.56" y="15.24" size="1.778" layer="95"/>
+</segment>
+</net>
+<net name="N$3" class="0">
+<segment>
+<pinref part="U1" gate="G$1" pin="XTAL1"/>
+<wire x1="-27.94" y1="0" x2="-38.1" y2="0" width="0.1524" layer="91"/>
+<wire x1="-38.1" y1="0" x2="-38.1" y2="5.08" width="0.1524" layer="91"/>
+<wire x1="-38.1" y1="5.08" x2="-43.18" y2="5.08" width="0.1524" layer="91"/>
+<pinref part="Q1" gate="G$1" pin="2"/>
+<wire x1="-43.18" y1="5.08" x2="-43.18" y2="2.54" width="0.1524" layer="91"/>
+</segment>
+</net>
+<net name="N$4" class="0">
+<segment>
+<pinref part="Q1" gate="G$1" pin="1"/>
+<wire x1="-43.18" y1="-7.62" x2="-43.18" y2="-10.16" width="0.1524" layer="91"/>
+<wire x1="-43.18" y1="-10.16" x2="-38.1" y2="-10.16" width="0.1524" layer="91"/>
+<wire x1="-38.1" y1="-10.16" x2="-38.1" y2="-2.54" width="0.1524" layer="91"/>
+<pinref part="U1" gate="G$1" pin="XTAL2"/>
+<wire x1="-38.1" y1="-2.54" x2="-27.94" y2="-2.54" width="0.1524" layer="91"/>
+</segment>
+</net>
 </nets>
 </sheet>
